File: pcb/PolyPot.sch (KiCad schematic (older format))
At the start: 25 parts

Commit message: Add temperature sensor, V_Bat sense
Parts:
- removed J?: PROG/DEBUG, symbol Conn_01x04
- removed J?: ANALOG_CONN, symbol Conn_01x04
- added C?: 100nF, symbol C
- added J?: ANALOG_CONN, symbol Conn_01x03
- added J?: V_BAT_1S, symbol Conn_01x02
- added J?: PROG/DEBUG, symbol Conn_01x06
- added TP? (x2): TEST, symbol TEST
- added U?: S-5851A_SOT-23-6, symbol S-5851A_SOT-23-6
- M?: value Motor_DC -> DC_WATER_PUMP
Connections:
- net labels added: PUMP_PWM, V_BAT_SENSE
- net labels removed: SENS_TEMP
- wire segments 45 -> 69
Other:
- note added: "Temperature sensor\naddress:\n0x48 (7bit)"
- moved on the sheet: C?, D?, JP?, M?, Q?, R?, SW?, TP?, U?

Commit message: Component annotation
Parts:
- gave numbers to parts that had none: 30

Commit message: Assign footprints, start with PCB
Parts:
- BT1, J1, JP1, JP2, M1: footprint (none) -> Socket_Strips:Socket_Strip_Straight_1x02_Pitch2.54mm
- C1, C2, C3, C4: footprint (none) -> Capacitors_SMD:C_0603_HandSoldering
- D1: footprint (none) -> LEDs:LED-3MM
- J2: footprint (none) -> Socket_Strips:Socket_Strip_Straight_1x06_Pitch2.54mm
- J3: footprint (none) -> Socket_Strips:Socket_Strip_Straight_1x03_Pitch2.54mm
- J4: footprint (none) -> Socket_Strips:Socket_Strip_Straight_1x05_Pitch2.54mm
- Q1, Q2: footprint (none) -> TO_SOT_Packages_SMD:SOT-23
- R1, R2, R3, R4, R5, R6: footprint (none) -> Resistors_SMD:R_0603_HandSoldering
- SW1, SW2: footprint (none) -> Buttons_Switches_SMD:SW_SPST_EVQPE1
- TP1, TP2, TP3, TP4: footprint (none) -> Socket_Strips:Socket_Strip_Straight_1x01
- U3: footprint (none) -> TO_SOT_Packages_SMD:SOT-23-6_Handsoldering
Connections:
- wire segments 69 -> 57

Commit message: Add ESP32 3d shape
Parts:
- U2: footprint ESP32-footprints-Lib:ESP32-WROOM -> PolyPot:ESP32-WROOM
Changed lines of the file:
@@
 F 0 "U2" H 3100 7050 60  0000 C CNN
 F 1 "ESP32-WROOM" H 4300 7050 60  0000 C CNN
-F 2 "ESP32-footprints-Lib:ESP32-WROOM" H 4150 7150 60  0001 C CNN
+F 2 "PolyPot:ESP32-WROOM" H 4150 7150 60  0001 C CNN
 F 3 "" H 3350 6250 60  0001 C CNN
 	1    3800 5800

Commit message: PCB: rough component placement
Parts:
- removed J1: V_BAT_1S, Socket_Strips:Socket_Strip_Straight_1x02_Pitch2.54mm, symbol Conn_01x02
- added J1: V_BAT_1S, Socket_Strips:Socket_Strip_Straight_1x01_Pitch2.54mm, symbol Conn_01x01
- added J5, J6, J7, J8: M3, Mounting_Holes:MountingHole_3.2mm_M3, symbol Conn_01x01
- D1: footprint LEDs:LED-3MM -> LEDs:LED_D3.0mm_Horizontal_O1.27mm_Z2.0mm
- J2: footprint Socket_Strips:Socket_Strip_Straight_1x06_Pitch2.54mm -> Socket_Strips:Socket_Strip_Straight_1x06_Pitch2.00mm
- J3: footprint Socket_Strips:Socket_Strip_Straight_1x03_Pitch2.54mm -> Socket_Strips:Socket_Strip_Straight_1x03_Pitch2.00mm
- J4: footprint Socket_Strips:Socket_Strip_Straight_1x05_Pitch2.54mm -> Socket_Strips:Socket_Strip_Straight_1x05_Pitch2.00mm
- JP1, JP2: footprint Socket_Strips:Socket_Strip_Straight_1x02_Pitch2.54mm -> Socket_Strips:Socket_Strip_Straight_1x02_Pitch1.27mm
- TP1, TP2, TP3, TP4: footprint Socket_Strips:Socket_Strip_Straight_1x01 -> Socket_Strips:Socket_Strip_Straight_1x01_Pitch1.27mm
Connections:
- wire segments 57 -> 56
- no-connect marks 0 -> 4
Other:
- note added: "Mounting holes"
Changed lines of the file:
@@
 F 0 "D1" H 3650 1500 50  0000 C CNN
 F 1 "LED" H 3650 1300 50  0000 C CNN
-F 2 "LEDs:LED-3MM" H 3650 1400 50  0001 C CNN
+F 2 "LEDs:LED_D3.0mm_Horizontal_O1.27mm_Z2.0mm" H 3650 1400 50  0001 C CNN
 F 3 "" H 3650 1400 50  0001 C CNN
 	1    3650 1400
@@
 F 0 "JP1" H 1550 1230 50  0000 C CNN
 F 1 "I_SENSE" H 1560 1090 50  0000 C CNN
-F 2 "Socket_Strips:Socket_Strip_Straight_1x02_Pitch2.54mm" H 1550 1150 50  0001 C CNN
+F 2 "Socket_Strips:Socket_Strip_Straight_1x02_Pitch1.27mm" H 1550 1150 50  0001 C CNN
 F 3 "" H 1550 1150 50  0001 C CNN
 	1    1550 1150
@@
 F 0 "TP2" H 7250 3500 50  0000 C BNN
 F 1 "TEST" H 7250 3450 50  0000 C CNN
-F 2 "Socket_Strips:Socket_Strip_Straight_1x01" H 7250 3200 50  0001 C CNN
+F 2 "Socket_Strips:Socket_Strip_Straight_1x01_Pitch1.27mm" H 7250 3200 50  0001 C CNN
 F 3 "" H 7250 3200 50  0001 C CNN
 	1    7250 3200
@@
 F 0 "TP1" H 7050 3650 50  0000 C BNN
 F 1 "TEST" H 7050 3600 50  0000 C CNN
-F 2 "Socket_Strips:Socket_Strip_Straight_1x01" H 7050 3350 50  0001 C CNN
+F 2 "Socket_Strips:Socket_Strip_Straight_1x01_Pitch1.27mm" H 7050 3350 50  0001 C CNN
 F 3 "" H 7050 3350 50  0001 C CNN
 	1    7050 3350
@@
 F 0 "JP2" H 7450 1630 50  0000 C CNN
 F 1 "I_SENSE" H 7460 1490 50  0000 C CNN
-F 2 "Socket_Strips:Socket_Strip_Straight_1x02_Pitch2.54mm" H 7450 1550 50  0001 C CNN
+F 2 "Socket_Strips:Socket_Strip_Straight_1x02_Pitch1.27mm" H 7450 1550 50  0001 C CNN
 F 3 "" H 7450 1550 50  0001 C CNN
 	1    7450 1550
@@
 F 0 "J4" H 10300 3350 50  0000 C CNN
 F 1 "TOF_DIST_SENS" H 10300 2750 50  0000 C CNN
-F 2 "Socket_Strips:Socket_Strip_Straight_1x05_Pitch2.54mm" H 10300 3050 50  0001 C CNN
+F 2 "Socket_Strips:Socket_Strip_Straight_1x05_Pitch2.00mm" H 10300 3050 50  0001 C CNN
 F 3 "" H 10300 3050 50  0001 C CNN
 	1    10300 3050
@@
 F 0 "J3" H 10300 2350 50  0000 C CNN
 F 1 "ANALOG_CONN" H 10300 1950 50  0000 C CNN
-F 2 "Socket_Strips:Socket_Strip_Straight_1x03_Pitch2.54mm" H 10300 2150 50  0001 C CNN
+F 2 "Socket_Strips:Socket_Strip_Straight_1x03_Pitch2.00mm" H 10300 2150 50  0001 C CNN
 F 3 "" H 10300 2150 50  0001 C CNN
 	1    10300 2150
@@
 F 0 "TP3" H 7700 5150 50  0000 C BNN
 F 1 "TEST" H 7700 5100 50  0000 C CNN
-F 2 "Socket_Strips:Socket_Strip_Straight_1x01" H 7700 4850 50  0001 C CNN
+F 2 "Socket_Strips:Socket_Strip_Straight_1x01_Pitch1.27mm" H 7700 4850 50  0001 C CNN
 F 3 "" H 7700 4850 50  0001 C CNN
 	1    7700 4850
@@
 F 0 "TP4" H 7700 6050 50  0000 C BNN
 F 1 "TEST" H 7700 6000 50  0000 C CNN
-F 2 "Socket_Strips:Socket_Strip_Straight_1x01" H 7700 5750 50  0001 C CNN
+F 2 "Socket_Strips:Socket_Strip_Straight_1x01_Pitch1.27mm" H 7700 5750 50  0001 C CNN
 F 3 "" H 7700 5750 50  0001 C CNN
 	1    7700 5750
@@
 Text Notes 9600 5850 0    60   ~ 0
 Temperature sensor\naddress:\n0x48 (7bit)
-$Comp
-L Conn_01x02 J1
-U 1 1 5A0486B1
-P 1450 2050
-F 0 "J1" H 1450 2150 50  0000 C CNN
-F 1 "V_BAT_1S" H 1450 1850 50  0000 C CNN
-F 2 "Socket_Strips:Socket_Strip_Straight_1x02_Pitch2.54mm" H 1450 2050 50  0001 C CNN
-F 3 "" H 1450 2050 50  0001 C CNN
-	1    1450 2050
-	1    0    0    -1
-$EndComp
-$Comp
-L GND #PWR021
-U 1 1 5A048EAB
-P 1050 2150
-F 0 "#PWR021" H 1050 1900 50  0001 C CNN
-F 1 "GND" H 1050 2000 50  0000 C CNN
-F 2 "" H 1050 2150 50  0001 C CNN
-F 3 "" H 1050 2150 50  0001 C CNN
-	1    1050 2150
-	1    0    0    -1
-$EndComp
-Wire Wire Line
-	1050 2150 1250 2150
 Text Label 650  2050 0    60   ~ 0
 V_BAT_SENSE
@@
 F 0 "J2" H 10300 1550 50  0000 C CNN
 F 1 "PROG/DEBUG" H 10300 850 50  0000 C CNN
-F 2 "Socket_Strips:Socket_Strip_Straight_1x06_Pitch2.54mm" H 10300 1250 50  0001 C CNN
+F 2 "Socket_Strips:Socket_Strip_Straight_1x06_Pitch2.00mm" H 10300 1250 50  0001 C CNN
 F 3 "" H 10300 1250 50  0001 C CNN
 	1    10300 1250
@@
 $EndComp
 $Comp
-L GND #PWR022
+L GND #PWR021
 U 1 1 5A04A9A0
 P 10850 4650
-F 0 "#PWR022" H 10850 4400 50  0001 C CNN
+F 0 "#PWR021" H 10850 4400 50  0001 C CNN
 F 1 "GND" H 10850 4500 50  0000 C CNN
 F 2 "" H 10850 4650 50  0001 C CNN
@@
 	10850 4200 10850 4350
 Connection ~ 10150 4200
+$Comp
+L Conn_01x01 J7
+U 1 1 5A046ABF
+P 6000 7350
+F 0 "J7" H 6000 7450 50  0000 C CNN
+F 1 "M3" H 6000 7250 50  0000 C CNN
+F 2 "Mounting_Holes:MountingHole_3.2mm_M3" H 6000 7350 50  0001 C CNN
+F 3 "" H 6000 7350 50  0001 C CNN
+	1    6000 7350
+	0    -1   -1   0
+$EndComp
+$Comp
+L Conn_01x01 J6
+U 1 1 5A046B30
+P 6300 7350
+F 0 "J6" H 6300 7450 50  0000 C CNN
+F 1 "M3" H 6300 7250 50  0000 C CNN
+F 2 "Mounting_Holes:MountingHole_3.2mm_M3" H 6300 7350 50  0001 C CNN
+F 3 "" H 6300 7350 50  0001 C CNN
+	1    6300 7350
+	0    -1   -1   0
+$EndComp
+$Comp
+L Conn_01x01 J5
+U 1 1 5A046BA2
+P 6600 7350
+F 0 "J5" H 6600 7450 50  0000 C CNN
+F 1 "M3" H 6600 7250 50  0000 C CNN
+F 2 "Mounting_Holes:MountingHole_3.2mm_M3" H 6600 7350 50  0001 C CNN
+F 3 "" H 6600 7350 50  0001 C CNN
+	1    6600 7350
+	0    -1   -1   0
+$EndComp
+Text Notes 5600 7200 0    60   ~ 0
+Mounting holes
+$Comp
+L Conn_01x01 J8
+U 1 1 5A0469DA
+P 5700 7350
+F 0 "J8" H 5700 7450 50  0000 C CNN
+F 1 "M3" H 5700 7250 50  0000 C CNN
+F 2 "Mounting_Holes:MountingHole_3.2mm_M3" H 5700 7350 50  0001 C CNN
+F 3 "" H 5700 7350 50  0001 C CNN
+	1    5700 7350
+	0    -1   -1   0
+$EndComp
+NoConn ~ 6600 7550
+NoConn ~ 6300 7550
+NoConn ~ 6000 7550
+NoConn ~ 5700 7550
+$Comp
+L Conn_01x01 J1
+U 1 1 5A049A8A
+P 1450 2050
+F 0 "J1" H 1450 2150 50  0000 C CNN
+F 1 "V_BAT_1S" H 1450 1950 50  0000 C CNN
+F 2 "Socket_Strips:Socket_Strip_Straight_1x01_Pitch2.54mm" H 1450 2050 50  0001 C CNN
+F 3 "" H 1450 2050 50  0001 C CNN
+	1    1450 2050
+	1    0    0    -1
+$EndComp
 $EndSCHEMATC
